File: Flight Controller.kicad_sch (KiCad schematic)
At the start: 146 parts, among them IC2 AT7456E, J1 Conn_01x08_MountingPin, J2 USB_C_Receptacle_USB2.0_14P, Q1 BC817W, U1 STM32F405RGTx, U2 LMR51430, U3 BMP280, U4 NCP1117-3.3_SOT223, U5 LMR51430, U6 W25Q128JVSIQ TR, U7 ICM-42688-P, U8 NCP1117-3.3_SOT223

Commit message: New connectors
Parts:
- removed TP_3V1: TestPoint, Connector:Soldier_Pad, symbol Connector:TestPoint
- added TP_10V1, TP_5V13: TestPoint, Connector:Soldier_Pad, symbol Connector:TestPoint
- R3, R4, R5, R6: value R -> 1k
Connections:
- net +10V: now also TP_10V1.1
- net +5V: now also TP_5V13.1
Other:
- moved on the sheet: TP_3V2, TP_5V5, TP_CAM1, TP_GND10, TP_GND11, TP_GND12, TP_GND13, TP_GND14, TP_GND6, TP_GND9, TP_RX3, TP_TX3

Commit message: New connectors
Parts:
- removed TP_10V1, TP_5V10, TP_5V8, TP_5V9, TP_GND10, TP_GND11, TP_GND12, TP_GND9, TP_RX6, TP_TX6: TestPoint, Connector:Soldier_Pad, symbol Connector:TestPoint
- added TP_10V2, TP_CC, TP_GND15, TP_TX1: TestPoint, Connector:Soldier_Pad, symbol Connector:TestPoint
- renumbered TP_SBUS1 to TP_RX1, TP_TX1 to TP_SBUS1
Connections:
- net +10V: now also TP_10V2.1
- net GND: now also TP_GND15.1
- net UART1_TX: now also TP_TX1.1
Other:
- note added: "Extra"
- note added: "GPS"
- note added: "Receiver"
- note removed: "Power"
- note removed: "UARTS"
- moved on the sheet: H1, H2, H3, H4, J1, R3_I2C1, R3_I2C2, TP_3V2, TP_5V11, TP_5V12, TP_5V13, TP_5V5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

Commit message: New connectors
Connections:
- net UART6_RX is gone; now on net S2: U1.38 (PC7)
- net UART6_TX is gone; now on net S1: U1.37 (PC6)
- net S1: no longer U1.42 (PA9)
- net S2: now also TP_S3.1; no longer TP_S2.1, U1.41 (PA8)
- net S3: now also TP_S2.1, U1.39 (PC8); no longer TP_S3.1, U1.40 (PC9)
- net S4: now also U1.40 (PC9); no longer U1.39 (PC8)
- no-connect marks 20 -> 22
Other:
- moved on the sheet: J1, R3_I2C1, R3_I2C2, TP_5V12, TP_Curr1, TP_GND14, TP_RX5, TP_Rssi1, TP_SCL1, TP_SDA1, TP_TX5, TP_VBAT1

Commit message: New connectors
Parts:
- removed R1, R2: 10k, Resistor_SMD:R_1206_3216Metric, symbol Device:R
- removed TP_Rssi1, TP_VBAT1: TestPoint, Connector:Soldier_Pad, symbol Connector:TestPoint
- added C6: 100n, Capacitor_SMD:C_0402_1005Metric, symbol Device:C
- added Q2: BC817W, Package_TO_SOT_SMD:SOT-323_SC-70, symbol Transistor_BJT:BC817W
- added R2_Buzzer: 1k, Resistor_SMD:R_0805_2012Metric, symbol Device:R
- added TP_GND9, TP_S5, TP_S6, TP_S7, TP_S8, TP_TEL: TestPoint, Connector:Soldier_Pad, symbol Connector:TestPoint
- added TP_VBAT+2: TestPoint, TestPoint:TestPoint_Pad_D2.5mm, symbol Connector:TestPoint
- added VBAT_R1: 100K, symbol Device:R
- added VBAT_R2: 10K, symbol Device:R
- JP1: value SolderJumper_3_Open -> Jumper_3
Connections:
- net +5V: now also TP_GND5.1
- net ADC_VBAT: now also C6.2, VBAT_R1.1, VBAT_R2.1
- net GND: now also C6.1, Q2.2 (E), TP_GND9.1, VBAT_R2.2; no longer TP_GND5.1
- net S1: now also TP_S5.1
- net S2: now also TP_S6.1
- net S3: now also TP_S7.1
- net S4: now also TP_S8.1
- net TEL: now also TP_TEL.1
- net VBAT+: now also TP_VBAT+2.1, VBAT_R1.2
- net NRST: now reaches C5.1, SW_NRST1.1, U1.7 (NRST)
- net CAP1: now reaches C1.2, U1.31 (VCAP_1)
- net CAP2: now reaches C2.2, U1.47 (VCAP_2)
- net RES1: now reaches 8M1.1, U1.5 (PH0)
- net RES2: now reaches 8M1.3, U1.6 (PH1)
- net BOOT: now reaches JP1.2 (C), U1.60 (BOOT0)
- net Beeper renamed BUZ
- net BUZ: now also R2_Buzzer.1
- net Buz renamed BUZ-
- net BUZ-: now also Q2.3 (C)
- new net: Q2.1 (B), R2_Buzzer.2
- no-connect marks 22 -> 23
Other:
- note added: "ADC Vbat"
- note added: "Boot Jumper"
- note added: "Caps"
- note added: "Chips"
- note added: "Microcontroller"
- note added: "NRST"
- note added: "Resonator"
- note removed: "Currents"
- note removed: "Sensors"
- moved on the sheet: 8M1, C1, C1_3R1, C1_3R2, C1_Dec1, C1_OSD1, C1out_5R1, C1out_5R2, C2, C2_3R1, C2_3R2, C2_Dec1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

Commit message: I hope I'm done here with the sch
Parts:
- added CC_R1: 220, symbol Device:R
- added D6: PESD1CANFD36LS-Q, Diode_SMD:D_SOD-882, symbol Device:D_TVS
- added J3: Conn_01x04, symbol Connector_Generic_MountingPin:Conn_01x04_MountingPin
- renumbered R2_Buzzer to Buzzer_R1
Connections:
- net I2C_SCL is gone; now on net I2C2_SCL: R3_I2C2.1, TP_SCL1.1
- net I2C_SDA is gone; now on net I2C2_SDA: R3_I2C1.2, TP_SDA1.1
- net LED_Out is gone; now on net LED_S: TP_LED1.1
- net +3.3V: now also J3.1 (Pin_1)
- net +5V: now also C1_3R1.1, C1_3R2.1, U4.3 (VI), U8.3 (VI)
- net 5V_OUT: no longer C1_3R1.1, C1_3R2.1, U4.3 (VI), U8.3 (VI)
- net GND: now also C1out_5R1.2, C1out_5R2.2, C2out_5R1.2, C2out_5R2.2, Cin2_5R1.2, Cin2_5R2.2, Cin3_5R1.1, Cin3_5R2.1, Cin_5R1.2, Cin_5R2.2, Rfbb_5R1.2, Rfbb_5R2.2, U2.1 (GND), U5.1 (GND), D6.2 (A2), J3.2 (Pin_2)
- net SWC: now also J3.4 (Pin_4)
- net SWD: now also J3.3 (Pin_3)
- net VBAT+: now also D6.1 (A1)
- net at TP_CC.1: now also CC_R1.2
- net LED_S: now reaches U1.41 (PA8)
- net CC: now reaches U1.42 (PA9)
- net CC: now also CC_R1.1
- net ADC_Rssi: no longer names the net of U1.10 (PC2)
Other:
- note added: "SWD"
- note added: "TVS"
- moved on the sheet: TP_10V2, TP_5V11, TP_5V5, TP_5V6, TP_CAM1, TP_CC, TP_GND13, TP_GND6, TP_GND7, TP_RX2, TP_RX3, TP_RX4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

Commit message: This time I'm done fr
Parts:
- removed C5: 100n, Capacitor_SMD:C_0402_1005Metric, symbol Device:C
- removed J3: Conn_01x04, symbol Connector_Generic_MountingPin:Conn_01x04_MountingPin
- removed SW_NRST1: SW_Push, Button_Switch_SMD:SW_Tactile_SPST_NO_Straight_CK_PTS636Sx25SMTRLFS, symbol Switch:SW_Push
- added BOOT_R1: 10k, symbol Device:R
- added TP_3V1, TP_GND10, TP_SWC1, TP_SWD1: TestPoint, Connector:Soldier_Pad, symbol Connector:TestPoint
- U1: value STM32F405RGTx -> AT32F435RGT7
- renumbered TP_CC to TP_CC1, TP_TEL to TP_TEL1
Connections:
- net +3.3V: now also TP_3V1.1
- net +5V: no longer C1_3R1.1, C1_3R2.1, U4.3 (VI), U8.3 (VI)
- net 5V_OUT: now also C1_3R1.1, C1_3R2.1, U4.3 (VI), U8.3 (VI)
- net BOOT: now also BOOT_R1.2; no longer JP1.2 (C)
- net GND: now also TP_GND10.1
- net GYRO_MISO: now also U1.35 (PB14); no longer U1.22 (PA6)
- net GYRO_MOSI: now also U1.36 (PB15); no longer U1.23 (PA7)
- net GYRO_SCLK: now also U1.34 (PB13); no longer U1.21 (PA5)
- net LED0: now also U1.26 (PB0); no longer U1.3 (PC14)
- net LED1: now also U1.27 (PB1); no longer U1.4 (PC15)
- net OSD_MISO: now also U1.22 (PA6); no longer U1.35 (PB14)
- net OSD_MOSI: now also U1.23 (PA7); no longer U1.36 (PB15)
- net OSD_SCLK: now also U1.21 (PA5); no longer U1.34 (PB13)
- net SWC: now also TP_SWC1.1
- net SWD: now also TP_SWD1.1
- net NRST: no longer names the net of U1.7 (NRST)
- new net: BOOT_R1.1, JP1.2 (C)
Other:
- note removed: "NRST"
- moved on the sheet: JP1, TP_10V2, TP_5V6, TP_GND13, TP_GND7, TP_RX2, TP_TX2, TP_VTX1

Commit message: I'm losing it
Changed lines of the file:
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@@
 	(text "Microcontroller"
 		(exclude_from_sim no)
-		(at 186.436 22.098 0)
+		(at 185.42 22.352 0)
 		(effects
 			(font
@@
 	(wire
 		(pts
-			(xy 97.79 242.57) (xy 97.79 245.11)
-		)
-		(stroke
-			(width 0)
-			(type default)
-		)
-	)
-	(wire
-		(pts
 			(xy 246.38 147.32) (xy 247.65 147.32)
 		)
@@
 	)
 	(symbol
-		(lib_id "power:PWR_FLAG")
-		(at 97.79 242.57 0)
-		(unit 1)
-		(exclude_from_sim no)
-		(in_bom yes)
-		(on_board yes)
-		(dnp no)
-		(property "Reference" "#FLG02"
-			(at 97.79 240.665 0)
-			(effects
-				(font
-					(size 1.27 1.27)
-				)
-				(hide yes)
-			)
-		)
-		(property "Value" "PWR_FLAG"
-			(at 97.79 238.76 0)
-			(effects
-				(font
-					(size 1.27 1.27)
-				)
-				(hide yes)
-			)
-		)
-		(property "Footprint" ""
-			(at 97.79 242.57 0)
-			(effects
-				(font
-					(size 1.27 1.27)
-				)
-				(hide yes)
-			)
-		)
-		(property "Datasheet" "~"
-			(at 97.79 242.57 0)
-			(effects
-				(font
-					(size 1.27 1.27)
-				)
-				(hide yes)
-			)
-		)
-		(property "Description" ""
-			(at 97.79 242.57 0)
-			(effects
-				(font
-					(size 1.27 1.27)
-				)
-			)
-		)
-		(pin "1"
-		)
-		(instances
-			(project "Flight Controller"
-				(path "/dbcd5f0a-1493-4b00-ba7e-2224e0d5072f"
-					(reference "#FLG02")
-					(unit 1)
-				)
-			)
-		)
-	)
-	(symbol
 		(lib_id "power:GND")
 		(at 83.82 175.26 270)
@@
 	)
 	(symbol
-		(lib_id "power:GND")
-		(at 97.79 245.11 0)
-		(unit 1)
-		(exclude_from_sim no)
-		(in_bom yes)
-		(on_board yes)
-		(dnp no)
-		(fields_autoplaced yes)
-		(property "Reference" "#PWR031"
-			(at 97.79 251.46 0)
-			(effects
-				(font
-					(size 1.27 1.27)
-				)
-				(hide yes)
-			)
-		)
-		(property "Value" "GND"
-			(at 97.79 250.19 0)
-			(effects
-				(font
-					(size 1.27 1.27)
-				)
-				(hide yes)
-			)
-		)
-		(property "Footprint" ""
-			(at 97.79 245.11 0)
-			(effects
-				(font
-					(size 1.27 1.27)
-				)
-				(hide yes)
-			)
-		)
-		(property "Datasheet" ""
-			(at 97.79 245.11 0)
-			(effects
-				(font
-					(size 1.27 1.27)
-				)
-				(hide yes)
-			)
-		)
-		(property "Description" ""
-			(at 97.79 245.11 0)
-			(effects
-				(font
-					(size 1.27 1.27)
-				)
-			)
-		)
-		(pin "1"
-		)
-		(instances
-			(project "Flight Controller"
-				(path "/dbcd5f0a-1493-4b00-ba7e-2224e0d5072f"
-					(reference "#PWR031")
-					(unit 1)
-				)
-			)
-		)
-	)
-	(symbol
 		(lib_id "Device:C")
 		(at 320.04 54.61 270)
@@
 				)
 				(justify left)
+				(hide yes)
 			)
 		)

Commit message: Updated naming system
Parts:
- C_3V1: renamed from C1_3R1; footprint Capacitor_SMD:C_0805_2012Metric -> Capacitor_SMD:C_0603_1608Metric
- C_3V2: renamed from C2_3R1; footprint Capacitor_SMD:C_0805_2012Metric -> Capacitor_SMD:C_0603_1608Metric
- C_3VG1: renamed from C1_3R2; footprint Capacitor_SMD:C_0805_2012Metric -> Capacitor_SMD:C_0603_1608Metric_Pad1.08x0.95mm_HandSolder
- C_3VG2: renamed from C2_3R2; footprint Capacitor_SMD:C_0805_2012Metric -> Capacitor_SMD:C_0603_1608Metric_Pad1.08x0.95mm_HandSolder
- C_DEC1: renamed from C1_Dec1; footprint Capacitor_SMD:C_0805_2012Metric -> Capacitor_SMD:C_0603_1608Metric
- C_GYRO1: renamed from C3_G1; footprint Capacitor_SMD:C_0805_2012Metric -> Capacitor_SMD:C_0402_1005Metric
- C_OSD2: renamed from C2_OSD1; footprint Capacitor_SMD:C_0805_2012Metric -> Capacitor_SMD:C_0402_1005Metric
- C_OSD3: renamed from C3_OSD1; footprint Capacitor_SMD:C_0805_2012Metric -> Capacitor_SMD:C_0402_1005Metric
- D_LED1: renamed from D1; footprint (none) -> LED_SMD:LED_0603_1608Metric
- D_LED2: renamed from D3; footprint (none) -> LED_SMD:LED_0603_1608Metric
- D_LED3: renamed from D4; footprint (none) -> LED_SMD:LED_0603_1608Metric
- D_LED4: renamed from D5; footprint (none) -> LED_SMD:LED_0603_1608Metric
- D_LED5: renamed from D1_LED1; footprint LED_SMD:LED_0402_1005Metric -> LED_SMD:LED_0603_1608Metric
- D_LED6: renamed from D2_LED1; footprint LED_SMD:LED_0402_1005Metric -> LED_SMD:LED_0603_1608Metric
- R_LED1: renamed from R3; footprint (none) -> Resistor_SMD:R_0603_1608Metric
- R_LED2: renamed from R4; footprint (none) -> Resistor_SMD:R_0603_1608Metric
- R_LED3: renamed from R5; footprint (none) -> Resistor_SMD:R_0603_1608Metric
- R_LED4: renamed from R6; footprint (none) -> Resistor_SMD:R_0603_1608Metric
- R_LED5: renamed from R1_LED1; footprint Resistor_SMD:R_0805_2012Metric -> Resistor_SMD:R_0603_1608Metric
- R_LED6: renamed from R2_LED1; footprint Resistor_SMD:R_0805_2012Metric -> Resistor_SMD:R_0603_1608Metric
- U6: footprint SOIC_208MIL_WIN -> (none)
- U7: footprint LGA14_2P5X3X0P91_TDK -> Package_LGA:Bosch_LGA-14_3x2.5mm_P0.5mm
- Y1: renamed from 8M1; value Resonator -> 8M
- renumbered Cboot_5R2 to CBOOT_10V1, Cboot_5R1 to CBOOT_5V1, Cin_5R2 to CIN_10V1, Cin2_5R2 to CIN_10V2, Cin3_5R2 to CIN_10V3, Cin_5R1 to CIN_5V1, Cin2_5R1 to CIN_5V2, Cin3_5R1 to CIN_5V3, C1out_5R2 to COUT_10V1, C2out_5R2 to COUT_10V2, C1out_5R1 to COUT_5V1, C2out_5R1 to COUT_5V2, C3 to C_BARO1, C4 to C_BARO2, C2_Dec1 to C_DEC2, C3_Dec1 to C_DEC3, C4_Dec1 to C_DEC4, C5_Dec1 to C_DEC5, C6_Dec1 to C_DEC6, C7_Dec1 to C_DEC7, C4_G1 to C_GYRO2, C2_G1 to C_GYRO3, C1_OSD1 to C_OSD1, C4_OSD1 to C_OSD4, C5_OSD1 to C_OSD5, C6_OSD1 to C_OSD6, C6 to C_VBAT1, L2 to L_10V1, L1 to L_5V1, Q1 to Q_SBUS1, Rfbb_5R2 to RFBB_10V1, Rfbb_5R1 to RFBB_5V1, Rfbt_5R2 to RFBT_10V1, Rfbt_5R1 to RFBT_5V1, BOOT_R1 to R_BOOT1, Buzzer_R1 to R_BUZ1, CC_R1 to R_CC1, FLASH_R1 to R_FLASH1, FLASH_R2 to R_FLASH2, R3_I2C1 to R_I2C1, R3_I2C2 to R_I2C2, R1_OSD1 to R_OSD1, R2_OSD1 to R_OSD2, R3_OSD1 to R_OSD3, R4_OSD1 to R_OSD4, R5_OSD1 to R_OSD5, R2_SBUS1 to R_SBUS1, R1_SBUS1 to R_SBUS2, R4_USB2 to R_USB1, R3_USB2 to R_USB2, VBAT_R1 to R_VBAT1, VBAT_R2 to R_VBAT2
Connections:
- net +3.3V: now also C_GYRO1.1, C_GYRO2.1, U7.8 (VDD)
- net +3.3V_GYRO: no longer C_GYRO1.1, C_GYRO2.1, U7.8 (VDD)
Other:
- moved on the sheet: C_GYRO1, C_GYRO2, R_USB1
