File: Flight Controller.kicad_sch (KiCad schematic)
At the start: 154 parts, among them IC2 AT7456E, J1 Conn_01x08_MountingPin, J2 USB_C_Receptacle_USB2.0_14P, Q2 BC817W, U1 AT32F435RGT7, U2 LMR51430, U3 BMP280, U4 NCP1117-3.3_SOT223, U5 LMR51430, U6 W25Q128JVSIQ TR, U7 ICM-42688-P, U8 NCP1117-3.3_SOT223, Y1 8M

Commit message: I'm losing it again
Parts:
- removed R_OSD3, R_OSD4, R_OSD5: 1k, Resistor_SMD:R_0805_2012Metric, symbol Device:R
- J1: footprint (none) -> Connector_JST:JST_SH_SM08B-SRSS-TB_1x08-1MP_P1.00mm_Horizontal
- R_BOOT1, R_CC1, R_FLASH1, R_FLASH2: footprint (none) -> Resistor_SMD:R_0402_1005Metric
- R_BUZ1: footprint Resistor_SMD:R_0805_2012Metric -> Resistor_SMD:R_0402_1005Metric
- R_I2C1, R_I2C2: footprint Resistor_SMD:R_0603_1608Metric -> Resistor_SMD:R_0402_1005Metric
- R_SBUS2: footprint Resistor_SMD:R_1206_3216Metric -> Resistor_SMD:R_0603_1608Metric
- R_VBAT1: footprint (none) -> Resistor_SMD:R_0805_2012Metric
- R_VBAT2: footprint (none) -> Resistor_SMD:R_1206_3216Metric
Connections:
- net CLKOUT: no longer names the net of IC2.7 (CLKOUT)
- net HS: no longer names the net of IC2.18 (~{HSYNC})
- net LOS: no longer names the net of IC2.12 (LOS)
- net VS: no longer names the net of IC2.17 (~{VSYNC})
- no-connect marks 23 -> 26
Other:
- moved on the sheet: C_OSD5, R_OSD2

Commit message: AHHHHHHHHHHHH
Parts:
- IC2: footprint MAX7456EUI:SOP65P637X110-28N -> max74:SOP65P637X110-28N
- J2: footprint Connector_USB:USB_C_Receptacle_HRO_TYPE-C-31-M-12 -> Connector_USB:USB_C_Receptacle_GCT_USB4110
- L_10V1: value 12.2u -> 12u; footprint Inductor_SMD:L_Abracon_ASPI-0630LR -> Inductor_SMD:L_Bourns_SRR1208_12.7x12.7mm
- L_5V1: value 8.6u -> 8.2u; footprint Inductor_SMD:L_Abracon_ASPI-0630LR -> Inductor_SMD:L_Vishay_IHLP-2525
- U6: footprint (none) -> footprints:SOIC_208MIL_WIN
Changed lines of the file:
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@@
 			)
 		)
-		(property "Value" "8.6u"
+		(property "Value" "8.2u"
 			(at 77.47 256.54 90)
 			(effects
@@
 			)
 		)
-		(property "Footprint" "Inductor_SMD:L_Abracon_ASPI-0630LR"
+		(property "Footprint" "Inductor_SMD:L_Vishay_IHLP-2525"
 			(at 77.47 255.27 0)
 			(effects
@@
 			)
 		)
-		(property "Footprint" "MAX7456EUI:SOP65P637X110-28N"
+		(property "Footprint" "max74:SOP65P637X110-28N"
 			(at 353.06 209.22 0)
 			(effects
@@
 			)
 		)
-		(property "Value" "12.2u"
+		(property "Value" "12u"
 			(at 186.69 256.54 90)
 			(effects
@@
 			)
 		)
-		(property "Footprint" "Inductor_SMD:L_Abracon_ASPI-0630LR"
+		(property "Footprint" "Inductor_SMD:L_Bourns_SRR1208_12.7x12.7mm"
 			(at 186.69 255.27 0)
 			(effects
@@
 			)
 		)
-		(property "Footprint" ""
+		(property "Footprint" "footprints:SOIC_208MIL_WIN"
 			(at 322.58 200.66 0)
 			(effects
@@
 			)
 		)
-		(property "Footprint" "Connector_USB:USB_C_Receptacle_HRO_TYPE-C-31-M-12"
+		(property "Footprint" "Connector_USB:USB_C_Receptacle_GCT_USB4110"
 			(at 36.83 156.21 0)
 			(effects

Commit message: One day this will be over
Parts:
- Y1: footprint Crystal:Resonator_SMD_Murata_CSTxExxV-3Pin_3.0x1.1mm -> (none)
- Y_OSD1: footprint Oscillator:Oscillator_SMD_Abracon_ASCO-4Pin_1.6x1.2mm -> (none)
Changed lines of the file:
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@@
 			)
 		)
-		(property "Footprint" "Oscillator:Oscillator_SMD_Abracon_ASCO-4Pin_1.6x1.2mm"
+		(property "Footprint" ""
 			(at 304.8 127 0)
 			(effects
@@
 			)
 		)
-		(property "Footprint" "Crystal:Resonator_SMD_Murata_CSTxExxV-3Pin_3.0x1.1mm"
+		(property "Footprint" ""
 			(at 195.58 36.195 0)
 			(effects

Commit message: Footprint Assignment Done
Parts:
- removed Y_OSD1: 27MHz, symbol Device:Crystal
- added Y2: 27M, AWSCR-27.00CV-T :E2X270061X04, symbol Device:Resonator
- Y1: footprint (none) -> Crystal:Resonator_SMD_Murata_CSTxExxV-3Pin_3.0x1.1mm
Connections:
- net GND: now also Y2.2
- net at IC2.5 (CLKIN): now also Y2.1
- net at IC2.6 (XFB): now also Y2.3
Changed lines of the file:
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@@
 	(wire
 		(pts
+			(xy 298.45 127) (xy 298.45 128.27)
+		)
+		(stroke
+			(width 0)
+			(type default)
+		)
+	)
+	(wire
+		(pts
 			(xy 113.03 165.1) (xy 114.3 165.1)
 		)
@@
 	(wire
 		(pts
+			(xy 298.45 127) (xy 299.72 127)
+		)
+		(stroke
+			(width 0)
+			(type default)
+		)
+	)
+	(wire
+		(pts
 			(xy 123.19 106.68) (xy 125.73 106.68)
 		)
@@
 	)
 	(symbol
-		(lib_id "Device:Crystal")
-		(at 304.8 127 270)
-		(unit 1)
-		(exclude_from_sim no)
-		(in_bom yes)
-		(on_board yes)
-		(dnp no)
-		(property "Reference" "Y_OSD1"
-			(at 297.18 123.444 90)
-			(effects
-				(font
-					(size 1.27 1.27)
-				)
-				(justify left)
-			)
-		)
-		(property "Value" "27MHz"
-			(at 297.18 129.54 90)
-			(effects
-				(font
-					(size 1.27 1.27)
-				)
-				(justify left)
-			)
-		)
-		(property "Footprint" ""
-			(at 304.8 127 0)
-			(effects
-				(font
-					(size 1.27 1.27)
-				)
-				(hide yes)
-			)
-		)
-		(property "Datasheet" "~"
-			(at 304.8 127 0)
-			(effects
-				(font
-					(size 1.27 1.27)
-				)
-				(hide yes)
-			)
-		)
-		(property "Description" ""
-			(at 304.8 127 0)
-			(effects
-				(font
-					(size 1.27 1.27)
-				)
-			)
-		)
-		(pin "2"
-		)
-		(pin "1"
-		)
-		(instances
-			(project "Flight Controller"
-				(path "/dbcd5f0a-1493-4b00-ba7e-2224e0d5072f"
-					(reference "Y_OSD1")
-					(unit 1)
-				)
-			)
-		)
-	)
-	(symbol
 		(lib_id "power:GND")
 		(at 232.41 55.88 0)
@@
 			)
 		)
-		(property "Footprint" ""
+		(property "Footprint" "Crystal:Resonator_SMD_Murata_CSTxExxV-3Pin_3.0x1.1mm"
 			(at 195.58 36.195 0)
 			(effects
@@
 	)
 	(symbol
+		(lib_id "Device:Resonator")
+		(at 304.8 127 270)
+		(unit 1)
+		(exclude_from_sim no)
+		(in_bom yes)
+		(on_board yes)
+		(dnp no)
+		(property "Reference" "Y2"
+			(at 301.244 132.588 90)
+			(effects
+				(font
+					(size 1.27 1.27)
+				)
+				(justify left)
+			)
+		)
+		(property "Value" "27M"
+			(at 300.736 121.666 90)
+			(effects
+				(font
+					(size 1.27 1.27)
+				)
+				(justify left)
+			)
+		)
+		(property "Footprint" "AWSCR-27.00CV-T :E2X270061X04"
+			(at 304.8 126.365 0)
+			(effects
+				(font
+					(size 1.27 1.27)
+				)
+				(hide yes)
+			)
+		)
+		(property "Datasheet" "~"
+			(at 304.8 126.365 0)
+			(effects
+				(font
+					(size 1.27 1.27)
+				)
+				(hide yes)
+			)
+		)
+		(property "Description" ""
+			(at 304.8 127 0)
+			(effects
+				(font
+					(size 1.27 1.27)
+				)
+			)
+		)
+		(pin "1"
+		)
+		(pin "2"
+		)
+		(pin "3"
+		)
+		(instances
+			(project "Flight Controller"
+				(path "/dbcd5f0a-1493-4b00-ba7e-2224e0d5072f"
+					(reference "Y2")
+					(unit 1)
+				)
+			)
+		)
+	)
+	(symbol
 		(lib_id "Device:R")
 		(at 251.46 238.76 90)
@@
 					(unit 1)
 				)
+			)
+		)
+	)
+	(symbol
+		(lib_id "power:GND")
+		(at 298.45 128.27 0)
+		(unit 1)
+		(exclude_from_sim no)
+		(in_bom yes)
+		(on_board yes)
+		(dnp no)
+		(fields_autoplaced yes)
+		(property "Reference" "#PWR028"
+			(at 298.45 134.62 0)
+			(effects
+				(font
+					(size 1.27 1.27)
+				)
+				(hide yes)
+			)
+		)
+		(property "Value" "GND"
+			(at 298.45 132.08 90)
+			(effects
+				(font
+					(size 1.27 1.27)
+				)
+				(justify right)
+				(hide yes)
+			)
+		)
+		(property "Footprint" ""
+			(at 298.45 128.27 0)
+			(effects
+				(font
+					(size 1.27 1.27)
+				)
+				(hide yes)
+			)
+		)
+		(property "Datasheet" ""
+			(at 298.45 128.27 0)
+			(effects
+				(font
+					(size 1.27 1.27)
+				)
+				(hide yes)
+			)
+		)
+		(property "Description" ""
+			(at 298.45 128.27 0)
+			(effects
+				(font
+					(size 1.27 1.27)
+				)
+			)
+		)
+		(pin "1"
+		)
+		(instances
+			(project "Flight Controller"
+				(path "/dbcd5f0a-1493-4b00-ba7e-2224e0d5072f"
+					(reference "#PWR028")
+					(unit 1)
+				)

Commit message: First Layout
Parts:
- CBOOT_10V1, CBOOT_5V1: footprint Capacitor_SMD:C_0402_1005Metric -> Capacitor_SMD:C_0603_1608Metric
- L_10V1: footprint Inductor_SMD:L_Bourns_SRR1208_12.7x12.7mm -> Wurth-Elektronik:744393465120
- RFBB_10V1, RFBB_5V1: footprint Resistor_SMD:R_0805_2012Metric -> Resistor_SMD:R_0402_1005Metric
- RFBT_10V1, RFBT_5V1: footprint Resistor_SMD:R_1206_3216Metric -> Resistor_SMD:R_0402_1005Metric
Connections:
- net +5V: now also D2.2; no longer D2.1
- net 5V_USB: now also D2.1; no longer D2.2
Changed lines of the file:
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@@
 	(wire
 		(pts
-			(xy 259.08 265.43) (xy 260.35 265.43)
-		)
-		(stroke
-			(width 0)
-			(type default)
-		)
-	)
-	(wire
-		(pts
 			(xy 132.08 83.82) (xy 133.35 83.82)
 		)
@@
 	(wire
 		(pts
+			(xy 241.3 265.43) (xy 243.84 265.43)
+		)
+		(stroke
+			(width 0)
+			(type default)
+		)
+	)
+	(wire
+		(pts
 			(xy 46.99 111.76) (xy 46.99 114.3)
 		)
@@
 	(wire
 		(pts
-			(xy 242.57 265.43) (xy 243.84 265.43)
-		)
-		(stroke
-			(width 0)
-			(type default)
-		)
-	)
-	(wire
-		(pts
 			(xy 31.75 278.13) (xy 25.4 278.13)
 		)
@@
 	(wire
 		(pts
+			(xy 259.08 265.43) (xy 262.89 265.43)
+		)
+		(stroke
+			(width 0)
+			(type default)
+		)
+	)
+	(wire
+		(pts
 			(xy 19.05 231.14) (xy 19.05 232.41)
 		)
@@
 	)
 	(label "5V_USB"
-		(at 260.35 265.43 0)
+		(at 241.3 265.43 180)
 		(effects
 			(font
 				(size 1.27 1.27)
 			)
-			(justify left bottom)
+			(justify right bottom)
 		)
 	)
@@
 			)
 		)
-		(property "Footprint" "Capacitor_SMD:C_0402_1005Metric"
+		(property "Footprint" "Capacitor_SMD:C_0603_1608Metric"
 			(at 180.34 254.3048 0)
 			(effects
@@
 			)
 		)
-		(property "Footprint" "Resistor_SMD:R_0805_2012Metric"
+		(property "Footprint" "Resistor_SMD:R_0402_1005Metric"
 			(at 82.042 270.51 90)
 			(effects
@@
 			)
 		)
-		(property "Footprint" "Resistor_SMD:R_1206_3216Metric"
+		(property "Footprint" "Resistor_SMD:R_0402_1005Metric"
 			(at 191.262 260.35 90)
 			(effects
@@
 			)
 		)
-		(property "Footprint" "Inductor_SMD:L_Bourns_SRR1208_12.7x12.7mm"
+		(property "Footprint" "Wurth-Elektronik:744393465120"
 			(at 186.69 255.27 0)
 			(effects
@@
 	(symbol
 		(lib_id "power:+5V")
-		(at 242.57 265.43 90)
+		(at 262.89 265.43 270)
 		(unit 1)
 		(exclude_from_sim no)
@@
 		(fields_autoplaced yes)
 		(property "Reference" "#PWR09"
-			(at 246.38 265.43 0)
+			(at 259.08 265.43 0)
 			(effects
 				(font
@@
 		)
 		(property "Value" "+5V"
-			(at 238.76 265.43 90)
+			(at 266.7 265.4299 90)
 			(effects
 				(font
@@
 		)
 		(property "Footprint" ""
-			(at 242.57 265.43 0)
+			(at 262.89 265.43 0)
 			(effects
 				(font
@@
 		)
 		(property "Datasheet" ""
-			(at 242.57 265.43 0)
+			(at 262.89 265.43 0)
 			(effects
 				(font
@@
 		)
 		(property "Description" ""
-			(at 242.57 265.43 0)
+			(at 262.89 265.43 0)
 			(effects
 				(font
@@
 			)
 		)
-		(property "Footprint" "Resistor_SMD:R_1206_3216Metric"
+		(property "Footprint" "Resistor_SMD:R_0402_1005Metric"
 			(at 82.042 260.35 90)
 			(effects
@@
 			)
 		)
-		(property "Footprint" "Capacitor_SMD:C_0402_1005Metric"
+		(property "Footprint" "Capacitor_SMD:C_0603_1608Metric"
 			(at 71.12 254.3048 0)
 			(effects
@@
 			)
 		)
-		(property "Footprint" "Resistor_SMD:R_0805_2012Metric"
+		(property "Footprint" "Resistor_SMD:R_0402_1005Metric"
 			(at 191.262 270.51 90)
 			(effects

Commit message: Updated Layout
Parts:
- TP_10V2, TP_3V1, TP_3V2, TP_5V1, TP_5V11, TP_5V12, TP_5V13, TP_5V2, TP_5V3, TP_5V4, TP_5V5, TP_5V6, TP_5V7, TP_Buz1, TP_CAM1, TP_CC1, TP_Curr1, TP_GND1, TP_GND10, TP_GND13, TP_GND14, TP_GND15, TP_GND2, TP_GND3, TP_GND4, TP_GND5, TP_GND6, TP_GND7, TP_GND8, TP_GND9, TP_LED1, TP_RX1, TP_RX2, TP_RX3, TP_RX4, TP_RX5, TP_S1, TP_S2, TP_S3, TP_S4, TP_S5, TP_S6, TP_S7, TP_S8, TP_SBUS1, TP_SCL1, TP_SDA1, TP_SWC1, TP_SWD1, TP_TEL1, TP_TX1, TP_TX2, TP_TX3, TP_TX4, TP_TX5, TP_VTX1: footprint Connector:Soldier_Pad -> Pads:Solder_Pad_SMD
- TP_VBAT+1, TP_VBAT+2, TP_VBAT-1: footprint TestPoint:TestPoint_Pad_D2.5mm -> Pads:Solder_Pad_SMD
Changed lines of the file:
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@@
 			)
 		)
-		(property "Footprint" "Connector:Soldier_Pad"
+		(property "Footprint" "Pads:Solder_Pad_SMD"
 			(at 133.35 77.47 0)
 			(effects
@@
 			)
 		)
-		(property "Footprint" "TestPoint:TestPoint_Pad_D2.5mm"
+		(property "Footprint" "Pads:Solder_Pad_SMD"
 			(at 114.3 151.13 0)
 			(effects
@@
 			)
 		)
-		(property "Footprint" "Connector:Soldier_Pad"
+		(property "Footprint" "Pads:Solder_Pad_SMD"
 			(at 107.95 81.28 0)
 			(effects
@@
 			)
 		)
-		(property "Footprint" "Connector:Soldier_Pad"
+		(property "Footprint" "Pads:Solder_Pad_SMD"
 			(at 154.94 130.81 0)
 			(effects
@@
 			)
 		)
-		(property "Footprint" "Connector:Soldier_Pad"
+		(property "Footprint" "Pads:Solder_Pad_SMD"
 			(at 85.09 171.45 0)
 			(effects
@@
 			)
 		)
-		(property "Footprint" "Connector:Soldier_Pad"
+		(property "Footprint" "Pads:Solder_Pad_SMD"
 			(at 158.75 86.36 0)
 			(effects
@@
 			)
 		)
-		(property "Footprint" "Connector:Soldier_Pad"
+		(property "Footprint" "Pads:Solder_Pad_SMD"
 			(at 85.09 162.56 0)
 			(effects
@@
 			)
 		)
-		(property "Footprint" "Connector:Soldier_Pad"
+		(property "Footprint" "Pads:Solder_Pad_SMD"
 			(at 86.36 114.3 0)
 			(effects
@@
 			)
 		)
-		(property "Footprint" "Connector:Soldier_Pad"
+		(property "Footprint" "Pads:Solder_Pad_SMD"
 			(at 160.02 167.64 0)
 			(effects
@@
 			)
 		)
-		(property "Footprint" "Connector:Soldier_Pad"
+		(property "Footprint" "Pads:Solder_Pad_SMD"
 			(at 158.75 115.57 0)
 			(effects
@@
 			)
 		)
-		(property "Footprint" "Connector:Soldier_Pad"
+		(property "Footprint" "Pads:Solder_Pad_SMD"
 			(at 85.09 168.91 0)
 			(effects
@@
 			)
 		)
-		(property "Footprint" "Connector:Soldier_Pad"
+		(property "Footprint" "Pads:Solder_Pad_SMD"
 			(at 114.3 168.91 0)
 			(effects
@@
 			)
 		)
-		(property "Footprint" "Connector:Soldier_Pad"
+		(property "Footprint" "Pads:Solder_Pad_SMD"
 			(at 85.09 189.23 0)
 			(effects
@@
 			)
 		)
-		(property "Footprint" "Connector:Soldier_Pad"
+		(property "Footprint" "Pads:Solder_Pad_SMD"
 			(at 158.75 113.03 0)
 			(effects
@@
 			)
 		)
-		(property "Footprint" "Connector:Soldier_Pad"
+		(property "Footprint" "Pads:Solder_Pad_SMD"
 			(at 133.35 82.55 0)
 			(effects
@@
 			)
 		)
-		(property "Footprint" "Connector:Soldier_Pad"
+		(property "Footprint" "Pads:Solder_Pad_SMD"
 			(at 114.3 166.37 0)
 			(effects
@@
 			)
 		)
-		(property "Footprint" "Connector:Soldier_Pad"
+		(property "Footprint" "Pads:Solder_Pad_SMD"
 			(at 158.75 88.9 0)
 			(effects
@@
 			)
 		)
-		(property "Footprint" "Connector:Soldier_Pad"
+		(property "Footprint" "Pads:Solder_Pad_SMD"
 			(at 85.09 184.15 0)
 			(effects
@@
 			)
 		)
-		(property "Footprint" "Connector:Soldier_Pad"
+		(property "Footprint" "Pads:Solder_Pad_SMD"
 			(at 154.94 133.35 0)
 			(effects
@@
 			)
 		)
-		(property "Footprint" "Connector:Soldier_Pad"
+		(property "Footprint" "Pads:Solder_Pad_SMD"
 			(at 158.75 110.49 0)
 			(effects
@@
 			)
 		)
-		(property "Footprint" "Connector:Soldier_Pad"
+		(property "Footprint" "Pads:Solder_Pad_SMD"
 			(at 90.17 120.65 0)
 			(effects
@@
 			)
 		)
-		(property "Footprint" "Connector:Soldier_Pad"
+		(property "Footprint" "Pads:Solder_Pad_SMD"
 			(at 83.82 91.44 0)
 			(effects
@@
 			)
 		)
-		(property "Footprint" "Connector:Soldier_Pad"
+		(property "Footprint" "Pads:Solder_Pad_SMD"
 			(at 158.75 71.12 0)
 			(effects
@@
 			)
 		)
-		(property "Footprint" "Connector:Soldier_Pad"
+		(property "Footprint" "Pads:Solder_Pad_SMD"
 			(at 85.09 175.26 0)
 			(effects
@@
 			)
 		)
-		(property "Footprint" "Connector:Soldier_Pad"
+		(property "Footprint" "Pads:Solder_Pad_SMD"
 			(at 85.09 86.36 0)
 			(effects
@@
 			)
 		)
-		(property "Footprint" "Connector:Soldier_Pad"
+		(property "Footprint" "Pads:Solder_Pad_SMD"
 			(at 154.94 135.89 0)
 			(effects
@@
 			)
 		)
-		(property "Footprint" "Connector:Soldier_Pad"
+		(property "Footprint" "Pads:Solder_Pad_SMD"
 			(at 86.36 106.68 0)
 			(effects
@@
 			)
 		)
-		(property "Footprint" "Connector:Soldier_Pad"
+		(property "Footprint" "Pads:Solder_Pad_SMD"
 			(at 114.3 161.29 0)
 			(effects
@@
 			)
 		)
-		(property "Footprint" "Connector:Soldier_Pad"
+		(property "Footprint" "Pads:Solder_Pad_SMD"
 			(at 158.75 107.95 0)
 			(effects
@@
 			)
 		)
-		(property "Footprint" "Connector:Soldier_Pad"
+		(property "Footprint" "Pads:Solder_Pad_SMD"
 			(at 85.09 83.82 0)
 			(effects
@@
 			)
 		)
-		(property "Footprint" "Connector:Soldier_Pad"
+		(property "Footprint" "Pads:Solder_Pad_SMD"
 			(at 109.22 77.47 0)
 			(effects
@@
 			)
 		)
-		(property "Footprint" "Connector:Soldier_Pad"
+		(property "Footprint" "Pads:Solder_Pad_SMD"
 			(at 133.35 85.09 0)
 			(effects
@@
 			)
 		)
-		(property "Footprint" "Connector:Soldier_Pad"
+		(property "Footprint" "Pads:Solder_Pad_SMD"
 			(at 160.02 165.1 0)
 			(effects
@@
 			)
 		)
-		(property "Footprint" "Connector:Soldier_Pad"
+		(property "Footprint" "Pads:Solder_Pad_SMD"
 			(at 109.22 86.36 0)
 			(effects
@@
 			)
 		)
-		(property "Footprint" "TestPoint:TestPoint_Pad_D2.5mm"
+		(property "Footprint" "Pads:Solder_Pad_SMD"
 			(at 82.55 140.97 0)
 			(effects
@@
 			)
 		)
-		(property "Footprint" "Connector:Soldier_Pad"
+		(property "Footprint" "Pads:Solder_Pad_SMD"
 			(at 114.3 153.67 0)
 			(effects
@@
 			)
 		)
-		(property "Footprint" "Connector:Soldier_Pad"
+		(property "Footprint" "Pads:Solder_Pad_SMD"
 			(at 86.36 111.76 0)
 			(effects
@@
 			)
 		)
-		(property "Footprint" "Connector:Soldier_Pad"
+		(property "Footprint" "Pads:Solder_Pad_SMD"
 			(at 158.75 91.44 0)
 			(effects
@@
 			)
 		)
-		(property "Footprint" "Connector:Soldier_Pad"
+		(property "Footprint" "Pads:Solder_Pad_SMD"
 			(at 86.36 109.22 0)
 			(effects
@@
 			)
 		)
-		(property "Footprint" "Connector:Soldier_Pad"
+		(property "Footprint" "Pads:Solder_Pad_SMD"
 			(at 85.09 180.34 0)
 			(effects
@@
 			)
 		)
-		(property "Footprint" "Connector:Soldier_Pad"
+		(property "Footprint" "Pads:Solder_Pad_SMD"
 			(at 158.75 74.93 0)
 			(effects
@@
 			)
 		)
-		(property "Footprint" "Connector:Soldier_Pad"
+		(property "Footprint" "Pads:Solder_Pad_SMD"
 			(at 133.35 87.63 0)
 			(effects
@@
 			)
 		)
-		(property "Footprint" "Connector:Soldier_Pad"
+		(property "Footprint" "Pads:Solder_Pad_SMD"
 			(at 85.09 88.9 0)
 			(effects
@@
 			)
 		)
-		(property "Footprint" "Connector:Soldier_Pad"
+		(property "Footprint" "Pads:Solder_Pad_SMD"
 			(at 109.22 83.82 0)
 			(effects
@@
 			)
 		)
-		(property "Footprint" "Connector:Soldier_Pad"
+		(property "Footprint" "Pads:Solder_Pad_SMD"
 			(at 133.35 74.93 0)
 			(effects
@@
 			)
 		)
-		(property "Footprint" "Connector:Soldier_Pad"
+		(property "Footprint" "Pads:Solder_Pad_SMD"
 			(at 85.09 177.8 0)
 			(effects
@@
 			)
 		)
-		(property "Footprint" "Connector:Soldier_Pad"
+		(property "Footprint" "Pads:Solder_Pad_SMD"
 			(at 114.3 163.83 0)
 			(effects
@@
 			)
 		)
-		(property "Footprint" "Connector:Soldier_Pad"
+		(property "Footprint" "Pads:Solder_Pad_SMD"
 			(at 154.94 138.43 0)
 			(effects
@@
 			)
 		)
-		(property "Footprint" "Connector:Soldier_Pad"
+		(property "Footprint" "Pads:Solder_Pad_SMD"
 			(at 85.09 166.37 0)
 			(effects
@@
 			)
 		)
-		(property "Footprint" "Connector:Soldier_Pad"
+		(property "Footprint" "Pads:Solder_Pad_SMD"
 			(at 133.35 80.01 0)
 			(effects
@@
 			)
 		)
-		(property "Footprint" "Connector:Soldier_Pad"
+		(property "Footprint" "Pads:Solder_Pad_SMD"
 			(at 85.09 186.69 0)
 			(effects
@@
 			)
 		)
-		(property "Footprint" "Connector:Soldier_Pad"
+		(property "Footprint" "Pads:Solder_Pad_SMD"
 			(at 85.09 160.02 0)
 			(effects
@@
 			)
 		)
-		(property "Footprint" "Connector:Soldier_Pad"
+		(property "Footprint" "Pads:Solder_Pad_SMD"
 			(at 86.36 116.84 0)
 			(effects
@@
 			)
 		)
-		(property "Footprint" "Connector:Soldier_Pad"
+		(property "Footprint" "Pads:Solder_Pad_SMD"
 			(at 158.75 105.41 0)
 			(effects
@@
 			)
 		)
-		(property "Footprint" "Connector:Soldier_Pad"
+		(property "Footprint" "Pads:Solder_Pad_SMD"
 			(at 114.3 158.75 0)
 			(effects
@@
 			)
 		)
-		(property "Footprint" "Connector:Soldier_Pad"
+		(property "Footprint" "Pads:Solder_Pad_SMD"
 			(at 114.3 156.21 0)
 			(effects
@@
 			)
 		)
-		(property "Footprint" "Connector:Soldier_Pad"
+		(property "Footprint" "Pads:Solder_Pad_SMD"
 			(at 158.75 102.87 0)
 			(effects
@@
 			)
 		)
-		(property "Footprint" "TestPoint:TestPoint_Pad_D2.5mm"
+		(property "Footprint" "Pads:Solder_Pad_SMD"
 			(at 82.55 138.43 0)
 			(effects
@@
 			)
 		)
-		(property "Footprint" "Connector:Soldier_Pad"
+		(property "Footprint" "Pads:Solder_Pad_SMD"
 			(at 85.09 157.48 0)
 			(effects

Commit message: Updated Layout
Connections:
- net LED0: now also U1.27 (PB1); no longer U1.26 (PB0)
- net LED1: now also U1.26 (PB0); no longer U1.27 (PB1)
Changed lines of the file:
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@@
 	)
 	(label "LED0"
-		(at 247.65 129.54 0)
+		(at 247.65 132.08 0)
 		(effects
 			(font
@@
 	)
 	(label "LED1"
-		(at 247.65 132.08 0)
-		(effects
-			(font
+		(at 247.65 129.54 0)
+		(effects
+			(font
