File: Flight Controller.kicad_pcb (KiCad board)
At the start: 4 copper layers, 39.5 x 39.5 mm, 95 parts, among them IC2 AT7456E, J1 Conn_01x08_MountingPin, J2 USB_C_Receptacle_USB2.0_14P, Q2 BC817W, U1 AT32F435RGT7, U2 LMR51430, U3 BMP280, U4 SPX3819M5-L-3-3, U5 LMR51430, U6 W25Q128JVSIQ TR, U7 ICM-42688-P, U8 SPX3819M5-L-3-3, Y1 8M, Y2 27M

Commit message: Layout Updates
Parts:
- added 10V: TestPoint, Pads:Solder_Pad_SMD, F.Cu at (137.0, 103.0)
- added 3.3V: TestPoint, Pads:Solder_Pad_SMD, F.Cu at (150.8, 70.3)
- added 3.3V: TestPoint, Pads:Solder_Pad_SMD, F.Cu at (146.8, 70.3)
- added 5V: TestPoint, Pads:Solder_Pad_SMD, F.Cu at (150.0, 99.5)
- added 5V: TestPoint, Pads:Solder_Pad_SMD, F.Cu at (141.8, 66.8)
- added 5V: TestPoint, Pads:Solder_Pad_SMD, F.Cu at (136.0, 99.5)
- added 5V: TestPoint, Pads:Solder_Pad_SMD, F.Cu at (145.8, 66.8)
- added 5V: TestPoint, Pads:Solder_Pad_SMD, F.Cu at (147.0, 103.0)
- added Buz: TestPoint, Pads:Solder_Pad_SMD, F.Cu at (151.8, 66.8)
- added CAM: TestPoint, Pads:Solder_Pad_SMD, F.Cu at (146.0, 99.5)
- added CC: TestPoint, Pads:Solder_Pad_SMD, F.Cu at (144.0, 99.5)
- added GND: TestPoint, Pads:Solder_Pad_SMD, F.Cu at (148.0, 99.5)
- added GND: TestPoint, Pads:Solder_Pad_SMD, F.Cu at (149.8, 66.8)
- added GND: TestPoint, Pads:Solder_Pad_SMD, F.Cu at (145.0, 103.0)
- added GND: TestPoint, Pads:Solder_Pad_SMD, F.Cu at (139.8, 66.8)
- added GND: TestPoint, Pads:Solder_Pad_SMD, F.Cu at (138.0, 99.5)
- added GND: TestPoint, Pads:Solder_Pad_SMD, F.Cu at (152.8, 70.3)
- added GND: TestPoint, Pads:Solder_Pad_SMD, F.Cu at (144.8, 70.3)
- added RX: TestPoint, Pads:Solder_Pad_SMD, F.Cu at (140.8, 70.3)
- added RX: TestPoint, Pads:Solder_Pad_SMD, F.Cu at (136.8, 70.3)
- added RX: TestPoint, Pads:Solder_Pad_SMD, F.Cu at (154.0, 99.5)
- added RX: TestPoint, Pads:Solder_Pad_SMD, F.Cu at (143.0, 103.0)
- added RX2: TestPoint, Pads:Solder_Pad_SMD, F.Cu at (140.0, 99.5)
- added SBUS: TestPoint, Pads:Solder_Pad_SMD, F.Cu at (143.8, 66.8)
- added SCL: TestPoint, Pads:Solder_Pad_SMD, F.Cu at (149.0, 103.0)
- added SDA: TestPoint, Pads:Solder_Pad_SMD, F.Cu at (151.0, 103.0)
- added SWC: TestPoint, Pads:Solder_Pad_SMD, F.Cu at (147.8, 66.8)
- added SWD: TestPoint, Pads:Solder_Pad_SMD, F.Cu at (148.8, 70.3)
- added TP_5V7: TestPoint, Pads:Solder_Pad_SMD, F.Cu at (169.7, 74.0)
- added TP_Curr1: TestPoint, Pads:Solder_Pad_SMD_Half, B.Cu at (139.6, 103.3)
- added TP_GND8: TestPoint, Pads:Solder_Pad_SMD, F.Cu at (171.6, 77.2)
- added TP_GND9: TestPoint, Pads:Solder_Pad_SMD_Half, B.Cu at (149.1, 103.3)
- added TP_LED1: TestPoint, Pads:Solder_Pad_SMD, F.Cu at (168.9, 77.2)
- added TP_S1: TestPoint, Pads:Solder_Pad_SMD_Half, B.Cu at (147.2, 103.3)
- added TP_S2: TestPoint, Pads:Solder_Pad_SMD_Half, B.Cu at (145.3, 103.3)
- added TP_S3: TestPoint, Pads:Solder_Pad_SMD_Half, B.Cu at (143.4, 103.3)
- added TP_S4: TestPoint, Pads:Solder_Pad_SMD_Half, B.Cu at (141.5, 103.3)
- added TP_TEL1: TestPoint, Pads:Solder_Pad_SMD_Half, B.Cu at (137.7, 103.3)
- added TP_VBAT+1: TestPoint, Pads:Solder_Pad_SMD, F.Cu at (56.4, 65.7)
- added TP_VBAT+2: TestPoint, Pads:Solder_Pad_SMD_Half, B.Cu at (151.0, 103.3)
- added TP_VBAT-1: TestPoint, Pads:Solder_Pad_SMD, F.Cu at (60.3, 54.4)
- added TX: TestPoint, Pads:Solder_Pad_SMD, F.Cu at (152.0, 99.5)
- added TX: TestPoint, Pads:Solder_Pad_SMD, F.Cu at (139.0, 103.0)
- added TX: TestPoint, Pads:Solder_Pad_SMD, F.Cu at (142.8, 70.3)
- added TX: TestPoint, Pads:Solder_Pad_SMD, F.Cu at (138.8, 70.3)
- added TX3: TestPoint, Pads:Solder_Pad_SMD, F.Cu at (142.0, 99.5)
- added VTX: TestPoint, Pads:Solder_Pad_SMD, F.Cu at (141.0, 103.0)
- moved G*** 19.5 mm to (161.3, 94.2)
- moved G*** 18.6 mm to (160.5, 110.7)
- moved G*** 10.9 mm to (142.3, 95.3)
- moved D6 2.50 mm to (147.2, 95.0)
- moved J1 2.50 mm to (144.3, 99.0)
- moved R_BUZ1 2.30 mm to (136.2, 76.5)
- moved Q2 1.97 mm to (139.5, 74.4)
- moved CBOOT_10V1 1.45 mm to (136.6, 87.9)
- moved CIN_10V2 1.24 mm to (136.3, 95.3)
- moved CIN_10V3 1.24 mm to (135.7, 97.0)
- moved U5 1.24 mm to (136.7, 90.4)
- moved CIN_10V1 1.24 mm to (136.3, 93.2)
- moved JP1 1.19 mm to (144.8, 74.5)
- moved R_BOOT1 1.19 mm to (144.9, 76.8)
- moved RFBB_10V1 0.89 mm to (140.4, 90.9)
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- renumbered D_LED2 to 10V, D_LED3 to 3.3V, D_LED4 to 3.3VGyro, D_LED1 to 5V, D_LED5 to FC1, D_LED6 to FC2
Routing:
- net /BUZ: track 14.4 -> 12.2 mm
- net Net-(Q2-B): track 2.08 -> 4.14 mm
- net Net-(D_LED1-A): track 3.14 -> 1.90 mm
- net /BOOT: track 3.28 -> 2.16 mm
- net Net-(D_LED4-A): track 3.04 -> 1.94 mm
- net Net-(D_LED2-A): track 3.14 -> 2.14 mm
- net Net-(D_LED5-A): track 3.04 -> 2.10 mm
- net Net-(D_LED6-A): track 3.04 -> 2.14 mm
- net Net-(D_LED3-A): track 3.14 -> 2.30 mm
Other:
- board text added: "Designed and Assembled in the Saudi Arabia"
