File: Flight Controller.kicad_pcb (KiCad board)
At the start: 4 copper layers, 39.5 x 39.5 mm, 142 parts, among them IC2 AT7456E, J1 Conn_01x08_MountingPin, J2 USB_C_Receptacle_USB2.0_14P, Q2 BC817W, U1 AT32F435RGT7, U2 LMR51430, U3 BMP280, U4 SPX3819M5-L-3-3, U5 LMR51430, U6 W25Q128JVSIQ TR, U7 ICM-42688-P, U8 SPX3819M5-L-3-3, Y1 8M, Y2 27M

Commit message: Layout Updates
Parts:
- moved TP_LED1 27.9 mm to (156.5, 52.2)
- moved TP_GND8 27.4 mm to (160.5, 52.2)
- moved 3.3V 26.1 mm to (149.6, 44.2)
- moved 3.3V 26.1 mm to (145.6, 44.2)
- moved 5V 26.1 mm to (140.6, 40.7)
- moved 5V 26.1 mm to (144.6, 40.7)
- moved Buz 26.1 mm to (150.6, 40.7)
- moved GND 26.1 mm to (148.6, 40.7)
- moved GND 26.1 mm to (138.6, 40.7)
- moved GND 26.1 mm to (151.6, 44.2)
- moved GND 26.1 mm to (143.6, 44.2)
- moved RX 26.1 mm to (139.6, 44.2)
- moved RX 26.1 mm to (135.6, 44.2)
- moved SBUS 26.1 mm to (142.6, 40.7)
- moved SWC 26.1 mm to (146.6, 40.7)
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Changed lines of the file:
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@@
 	(footprint "Pads:Solder_Pad_SMD"
 		(layer "F.Cu")
-		(at 168.9 77.2)
+		(at 156.5 52.2)
 		(descr "solder Pin_ diameter 1.0mm, hole diameter 1.0mm (press fit), length 10.0mm")
 		(tags "solder Pin_ press fit")
@@
 	(footprint "Pads:Solder_Pad_SMD"
 		(layer "F.Cu")
-		(at 150.8 70.3 180)
+		(at 149.6 44.2 180)
 		(descr "solder Pin_ diameter 1.0mm, hole diameter 1.0mm (press fit), length 10.0mm")
 		(tags "solder Pin_ press fit")
@@
 	(footprint "Pads:Solder_Pad_SMD"
 		(layer "F.Cu")
-		(at 169.65 73.95)
+		(at 158.5 52.2)
 		(descr "solder Pin_ diameter 1.0mm, hole diameter 1.0mm (press fit), length 10.0mm")
 		(tags "solder Pin_ press fit")
@@
 	(footprint "Pads:Solder_Pad_SMD"
 		(layer "F.Cu")
-		(at 143.8 66.8 180)
+		(at 142.6 40.7 180)
 		(descr "solder Pin_ diameter 1.0mm, hole diameter 1.0mm (press fit), length 10.0mm")
 		(tags "solder Pin_ press fit")
@@
 	(footprint "Pads:Solder_Pad_SMD"
 		(layer "F.Cu")
-		(at 141.8 66.8 180)
+		(at 140.6 40.7 180)
 		(descr "solder Pin_ diameter 1.0mm, hole diameter 1.0mm (press fit), length 10.0mm")
 		(tags "solder Pin_ press fit")
@@
 	(footprint "Pads:Solder_Pad_SMD"
 		(layer "F.Cu")
-		(at 151.8 66.8 180)
+		(at 150.6 40.7 180)
 		(descr "solder Pin_ diameter 1.0mm, hole diameter 1.0mm (press fit), length 10.0mm")
 		(tags "solder Pin_ press fit")
@@
 	(footprint "Pads:Solder_Pad_SMD"
 		(layer "F.Cu")
-		(at 147.8 66.8 180)
+		(at 146.6 40.7 180)
 		(descr "solder Pin_ diameter 1.0mm, hole diameter 1.0mm (press fit), length 10.0mm")
 		(tags "solder Pin_ press fit")
@@
 	(footprint "Pads:Solder_Pad_SMD"
 		(layer "F.Cu")
-		(at 149.8 66.8 180)
+		(at 148.6 40.7 180)
 		(descr "solder Pin_ diameter 1.0mm, hole diameter 1.0mm (press fit), length 10.0mm")
 		(tags "solder Pin_ press fit")
@@
 	(footprint "Pads:Solder_Pad_SMD"
 		(layer "F.Cu")
-		(at 140.8 70.3 180)
+		(at 139.6 44.2 180)
 		(descr "solder Pin_ diameter 1.0mm, hole diameter 1.0mm (press fit), length 10.0mm")
 		(tags "solder Pin_ press fit")
@@
 	(footprint "Pads:Solder_Pad_SMD"
 		(layer "F.Cu")
-		(at 146.8 70.3 180)
+		(at 145.6 44.2 180)
 		(descr "solder Pin_ diameter 1.0mm, hole diameter 1.0mm (press fit), length 10.0mm")
 		(tags "solder Pin_ press fit")
@@
 	(footprint "Pads:Solder_Pad_SMD"
 		(layer "F.Cu")
-		(at 171.6 77.25)
+		(at 160.5 52.2)
 		(descr "solder Pin_ diameter 1.0mm, hole diameter 1.0mm (press fit), length 10.0mm")
 		(tags "solder Pin_ press fit")
@@
 	(footprint "Pads:Solder_Pad_SMD"
 		(layer "F.Cu")
-		(at 142.8 70.3 180)
+		(at 141.6 44.2 180)
 		(descr "solder Pin_ diameter 1.0mm, hole diameter 1.0mm (press fit), length 10.0mm")
 		(tags "solder Pin_ press fit")
@@
 	(footprint "Pads:Solder_Pad_SMD"
 		(layer "F.Cu")
-		(at 136.8 70.3 180)
+		(at 135.6 44.2 180)
 		(descr "solder Pin_ diameter 1.0mm, hole diameter 1.0mm (press fit), length 10.0mm")
 		(tags "solder Pin_ press fit")
@@
 	(footprint "Pads:Solder_Pad_SMD"
 		(layer "F.Cu")
-		(at 139.8 66.8 180)
+		(at 138.6 40.7 180)
 		(descr "solder Pin_ diameter 1.0mm, hole diameter 1.0mm (press fit), length 10.0mm")
 		(tags "solder Pin_ press fit")
@@
 	(footprint "Pads:Solder_Pad_SMD"
 		(layer "F.Cu")
-		(at 138.8 70.3 180)
+		(at 137.6 44.2 180)
 		(descr "solder Pin_ diameter 1.0mm, hole diameter 1.0mm (press fit), length 10.0mm")
 		(tags "solder Pin_ press fit")
@@
 	(footprint "Pads:Solder_Pad_SMD"
 		(layer "F.Cu")
-		(at 152.8 70.3 180)
+		(at 151.6 44.2 180)
 		(descr "solder Pin_ diameter 1.0mm, hole diameter 1.0mm (press fit), length 10.0mm")
 		(tags "solder Pin_ press fit")
@@
 	(footprint "Pads:Solder_Pad_SMD"
 		(layer "F.Cu")
-		(at 145.8 66.8 180)
+		(at 144.6 40.7 180)
 		(descr "solder Pin_ diameter 1.0mm, hole diameter 1.0mm (press fit), length 10.0mm")
 		(tags "solder Pin_ press fit")
@@
 	(footprint "Pads:Solder_Pad_SMD"
 		(layer "F.Cu")
-		(at 144.8 70.3 180)
+		(at 143.6 44.2 180)
 		(descr "solder Pin_ diameter 1.0mm, hole diameter 1.0mm (press fit), length 10.0mm")
 		(tags "solder Pin_ press fit")
@@
 	(footprint "Pads:Solder_Pad_SMD"
 		(layer "F.Cu")
-		(at 148.8 70.3 180)
+		(at 147.6 44.2 180)
 		(descr "solder Pin_ diameter 1.0mm, hole diameter 1.0mm (press fit), length 10.0mm")
 		(tags "solder Pin_ press fit")

Commit message: Layout Updates
Parts:
- removed JP1: Jumper_3, Jumper:SolderJumper-3_P1.3mm_Open_Pad1.0x1.5mm_NumberLabels
- added SW1: SW_SPST, Button_Switch_SMD:SW_SPST_EVQP2_MiddlePushTravel_H2.5mm, F.Cu at (145.8, 74.3)
- added TP_5V1: TestPoint, Pads:Solder_Pad_SMD, F.Cu at (133.2, 66.8)
- added TP_5V2: TestPoint, Pads:Solder_Pad_SMD, F.Cu at (153.2, 103.5)
- added TP_5V3: TestPoint, Pads:Solder_Pad_SMD, F.Cu at (133.2, 103.5)
- added TP_GND1: TestPoint, Pads:Solder_Pad_SMD, F.Cu at (135.0, 66.8)
- added TP_GND2: TestPoint, Pads:Solder_Pad_SMD, F.Cu at (155.0, 103.5)
- added TP_GND3: TestPoint, Pads:Solder_Pad_SMD, F.Cu at (135.0, 103.5)
- added TP_LED2: TestPoint, Pads:Solder_Pad_SMD, F.Cu at (136.8, 66.8)
- added TP_LED3: TestPoint, Pads:Solder_Pad_SMD, F.Cu at (156.8, 103.5)
- added TP_LED4: TestPoint, Pads:Solder_Pad_SMD, F.Cu at (136.8, 103.5)
- moved TP_Buz1 29.7 mm to (147.2, 70.2)
- moved TP_GND5 29.7 mm to (145.5, 70.2)
- moved TP_SWC1 29.7 mm to (143.8, 70.2)
- moved TP_5V13 29.7 mm to (142.0, 70.2)
- moved TP_SBUS1 29.6 mm to (140.2, 70.2)
- moved TP_5V11 29.6 mm to (138.5, 70.2)
- moved TP_GND13 29.6 mm to (136.8, 70.2)
- moved TP_SWD1 26.1 mm to (149.0, 70.2)
- moved TP_3V1 26.1 mm to (150.8, 70.2)
- moved TP_GND10 26.1 mm to (152.5, 70.2)
- moved TP_RX4 23.2 mm to (141.0, 66.8)
- moved TP_TX4 23.1 mm to (142.8, 66.8)
- moved TP_RX1 23.1 mm to (144.5, 66.8)
- moved TP_TX1 23.0 mm to (146.2, 66.8)
- moved TP_GND15 23.0 mm to (148.0, 66.8)
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- renumbered 10V to TP_10V2, 3.3V to TP_3V1, 3.3V to TP_3V2, 5V to TP_5V11, 5V to TP_5V12, 5V to TP_5V13, 5V to TP_5V5, 5V to TP_5V6, Buz to TP_Buz1, CAM to TP_CAM1, CC to TP_CC1, GND to TP_GND10, GND to TP_GND13, GND to TP_GND14, GND to TP_GND15, GND to TP_GND5, GND to TP_GND6, GND to TP_GND7, RX to TP_RX1, RX2 to TP_RX2, RX to TP_RX3, RX to TP_RX4, RX to TP_RX5, SBUS to TP_SBUS1, SCL to TP_SCL1, SDA to TP_SDA1, SWC to TP_SWC1, SWD to TP_SWD1, TX to TP_TX1, TX to TP_TX2, TX3 to TP_TX3, TX to TP_TX4, TX to TP_TX5, VTX to TP_VTX1
Connections:
- R_BOOT1 pad 1: Net-(JP1-C) -> GND
Routing:
- net /UART5_TX: track 0.00 -> 50.7 mm, vias 0 -> 2
- net /UART5_RX: track 0.00 -> 37.9 mm, vias 0 -> 4
- net /UART3_RX: track 0.00 -> 30.6 mm, vias 0 -> 4
- net /UART3_TX: track 0.00 -> 30.2 mm, vias 0 -> 2
- net /UART2_TX: track 0.00 -> 20.1 mm
- net /UART2_RX: track 0.00 -> 13.4 mm
- net /I2C2_SCL: track 3.23 -> 13.4 mm, vias 0 -> 2
- net /BOOT: track 2.16 -> 11.3 mm
- net /I2C2_SDA: track 2.67 -> 10.7 mm, vias 0 -> 2
- net +3.3V: track 16.7 -> 21.8 mm
- net /GYRO_INT: track 10.7 -> 12.5 mm
- net Net-(JP1-C): track 1.76 -> 0.00 mm
- net /UART1_TX: track 12.1 -> 13.2 mm
- net /GYRO_CS: track 15.1 -> 16.0 mm

Commit message: Layout Updates
Parts:
- renumbered TP_10V2 to 10V, TP_5V12 to 5V, TP_5V6 to 5V, TP_5V3 to 5V, TP_5V2 to 5V, TP_5V1 to 5V, TP_5V5 to 5V, TP_CAM1 to CAM, TP_CC1 to CC, TP_GND14 to GND, TP_GND10 to GND, TP_GND15 to GND, TP_GND1 to GND, TP_GND3 to GND, TP_GND5 to GND, TP_GND6 to GND, TP_GND2 to GND, TP_GND8 to GND, TP_GND13 to GND, TP_GND7 to GND, TP_LED4 to LED, TP_LED3 to LED, TP_LED2 to LED, TP_RX2 to RX2, TP_RX3 to RX3, TP_RX5 to RX5, TP_SCL1 to SCL, TP_SDA1 to SDA, TP_TX2 to TX2, TP_TX3 to TX3, TP_TX5 to TX5, TP_VTX1 to VTX
Routing:
- net /UART3_TX: track 30.2 -> 40.7 mm
- net /UART3_RX: track 30.6 -> 33.6 mm

Commit message: Layout Updates
Parts:
- moved TP_5V5 60.8 mm to (145.4, 39.2)
- moved TP_CAM1 60.8 mm to (149.2, 42.7)
- moved TP_CC1 60.8 mm to (141.9, 39.2)
- moved TP_GND6 60.8 mm to (143.7, 39.2)
- moved TP_RX3 60.8 mm to (147.4, 42.7)
- moved TP_TX3 60.8 mm to (145.7, 42.7)
- moved TP_5V11 44.7 mm to (135.5, 114.8)
- moved TP_GND13 44.7 mm to (133.8, 114.8)
- moved TP_RX4 44.7 mm to (138.0, 111.3)
- moved TP_TX4 44.7 mm to (139.8, 111.3)
- moved TP_3V1 44.5 mm to (155.0, 114.5)
- moved TP_GND10 44.5 mm to (156.8, 114.5)
- moved TP_SWC1 44.5 mm to (148.0, 114.5)
- moved TP_SWD1 44.5 mm to (153.2, 114.5)
- moved TP_VBAT+1 37.6 mm to (93.6, 60.0)
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- renumbered 5V to D_LED1, 10V to D_LED2, 3.3V to D_LED3, 3.3VGyro to D_LED4, FC1 to D_LED5, FC2 to D_LED6, 10V to TP_10V2, 5V to TP_5V1, 5V to TP_5V12, 5V to TP_5V2, 5V to TP_5V3, 5V to TP_5V5, 5V to TP_5V6, CAM to TP_CAM1, CC to TP_CC1, GND to TP_GND1, GND to TP_GND10, GND to TP_GND13, GND to TP_GND14, GND to TP_GND15, GND to TP_GND2, GND to TP_GND3, GND to TP_GND5, GND to TP_GND6, GND to TP_GND7, GND to TP_GND8, LED to TP_LED2, LED to TP_LED3, LED to TP_LED4, RX2 to TP_RX2, RX3 to TP_RX3, RX5 to TP_RX5, SCL to TP_SCL1, SDA to TP_SDA1, TX2 to TP_TX2, TX3 to TP_TX3, TX5 to TP_TX5, VTX to TP_VTX1
Routing:
- net /UART5_TX: track 50.7 -> 0.00 mm, vias 2 -> 0
- net /UART3_TX: track 40.7 -> 0.00 mm, vias 2 -> 0
- net /UART5_RX: track 37.9 -> 0.00 mm, vias 4 -> 0
- net /UART3_RX: track 33.6 -> 0.00 mm, vias 4 -> 0
- net /FLASH_CS: track 33.4 -> 0.00 mm, vias 1 -> 0
- net /UART2_TX: track 20.1 -> 0.00 mm
- net /OSD_MISO: track 19.3 -> 0.00 mm, vias 3 -> 0
- net /OSD_SCLK: track 18.6 -> 0.00 mm, vias 3 -> 0
- net /GYRO_CS: track 16.0 -> 0.00 mm, vias 2 -> 0
- net /FLASH_MISO: track 13.6 -> 0.00 mm, vias 1 -> 0
- net /UART2_RX: track 13.4 -> 0.00 mm
- net /GYRO_INT: track 12.5 -> 0.00 mm
- net /FLASH_MOSI: track 14.1 -> 1.64 mm
- net /OSD_CS: track 12.1 -> 0.00 mm, vias 1 -> 0
- net /FLASH_SCLK: track 11.2 -> 0.00 mm, vias 1 -> 0
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
Commit message: Layout Updates
Parts:
- moved TP_5V5 61.3 mm to (153.5, 100.0)
- moved TP_CC1 61.3 mm to (150.0, 100.0)
- moved TP_GND6 61.3 mm to (151.8, 100.0)
- moved TP_CAM1 60.8 mm to (147.5, 103.5)
- moved TP_RX3 60.8 mm to (145.8, 103.5)
- moved TP_TX3 60.8 mm to (144.0, 103.5)
- moved TP_5V11 48.3 mm to (154.2, 70.2)
- moved TP_GND13 48.3 mm to (152.5, 70.2)
- moved TP_3V1 46.1 mm to (142.0, 70.2)
- moved TP_GND10 46.1 mm to (143.8, 70.2)
- moved TP_SWD1 46.1 mm to (140.2, 70.2)
- moved TP_SWC1 45.3 mm to (138.5, 70.2)
- moved TP_RX4 42.5 mm to (149.0, 70.2)
- moved TP_TX4 42.5 mm to (150.8, 70.2)
- moved TP_10V2 33.3 mm to (138.8, 103.5)
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Routing:
- net /OSD_SCLK: track 0.00 -> 24.0 mm, vias 0 -> 1
- net /OSD_MOSI: track 0.00 -> 21.8 mm, vias 0 -> 1
- net /FLASH_MISO: track 0.00 -> 17.3 mm, vias 0 -> 1
- net /OSD_MISO: track 0.00 -> 17.2 mm, vias 0 -> 1
- net /OSD_CS: track 0.00 -> 15.2 mm, vias 0 -> 1
- net /FLASH_SCLK: track 0.00 -> 14.3 mm, vias 0 -> 1
- net /FLASH_MOSI: track 1.64 -> 8.30 mm
- net Net-(IC2-CLKIN): track 0.00 -> 5.20 mm
- net Net-(IC2-XFB): track 0.00 -> 3.16 mm
- net /CC: track 1.62 -> 0.00 mm
- net /ADC_VBAT: track 6.15 -> 4.78 mm

Commit message: We are going 6 layers BABYYgit add --all!
Parts:
- FC 1: renamed from D_LED5
- FC 2: renamed from D_LED6
- renumbered D_LED2 to 10V, TP_10V2 to 10V, D_LED3 to 3.3V, D_LED4 to 3.3VG, TP_5V12 to 5V, TP_5V6 to 5V, TP_5V3 to 5V, D_LED1 to 5V, TP_5V2 to 5V, TP_5V5 to 5V, TP_CAM1 to CAM, TP_CC1 to CC, TP_GND14 to GND, TP_GND3 to GND, TP_GND6 to GND, TP_GND2 to GND, TP_GND7 to GND, TP_LED4 to LED, TP_LED3 to LED, TP_RX2 to RX2, TP_RX3 to RX3, TP_RX5 to RX5, TP_SCL1 to SCL, TP_SDA1 to SDA, TP_TX2 to TX2, TP_TX3 to TX3, TP_TX5 to TX5, TP_VTX1 to VTX
Other:
- copper layers 4 -> 6
Changed lines of the file:
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@@
 	(generator_version "9.0")
 	(general
-		(thickness 1.6)
+		(thickness 1.566)
 		(legacy_teardrops no)
 	)
@@
 		(0 "F.Cu" signal)
 		(4 "In1.Cu" power)
-		(6 "In2.Cu" power)
+		(6 "In2.Cu" signal)
+		(8 "In3.Cu" power)
+		(10 "In4.Cu" power)
 		(2 "B.Cu" signal)
 		(9 "F.Adhes" user "F.Adhesive")
@@
 			(layer "dielectric 1"
 				(type "prepreg")
-				(thickness 0.1)
+				(thickness 0.0994)
 				(material "FR4")
 				(epsilon_r 4.5)
@@
 			(layer "In1.Cu"
 				(type "copper")
-				(thickness 0.035)
+				(thickness 0.0152)
 			)
 			(layer "dielectric 2"
 				(type "core")
-				(thickness 1.24)
+				(thickness 0.55)
 				(material "FR4")
 				(epsilon_r 4.5)
@@
 			(layer "In2.Cu"
 				(type "copper")
-				(thickness 0.035)
+				(thickness 0.0152)
 			)
 			(layer "dielectric 3"
 				(type "prepreg")
-				(thickness 0.1)
+				(thickness 0.1164)
+				(material "FR4")
+				(epsilon_r 4.5)
+				(loss_tangent 0.02)
+			)
+			(layer "In3.Cu"
+				(type "copper")
+				(thickness 0.0152)
+			)
+			(layer "dielectric 4"
+				(type "core")
+				(thickness 0.55)
+				(material "FR4")
+				(epsilon_r 4.5)
+				(loss_tangent 0.02)
+			)
+			(layer "In4.Cu"
+				(type "copper")
+				(thickness 0.0152)
+			)
+			(layer "dielectric 5"
+				(type "prepreg")
+				(thickness 0.0994)
 				(material "FR4")
 				(epsilon_r 4.5)
@@
 		(descr "solder Pin_ diameter 1.0mm, hole diameter 1.0mm (press fit), length 10.0mm")
 		(tags "solder Pin_ press fit")
-		(property "Reference" "TP_LED4"
+		(property "Reference" "LED"
 			(at -0.05 -1.4 0)
 			(layer "F.SilkS")
@@
 		(descr "solder Pin_ diameter 1.0mm, hole diameter 1.0mm (press fit), length 10.0mm")
 		(tags "solder Pin_ press fit")
-		(property "Reference" "TP_TX5"
+		(property "Reference" "TX5"
 			(at 0.05 -1.4 0)
 			(layer "F.SilkS")
@@
 		(descr "solder Pin_ diameter 1.0mm, hole diameter 1.0mm (press fit), length 10.0mm")
 		(tags "solder Pin_ press fit")
-		(property "Reference" "TP_5V12"
+		(property "Reference" "5V"
 			(at 0.05 -1.4 0)
 			(layer "F.SilkS")
@@
 		(descr "solder Pin_ diameter 1.0mm, hole diameter 1.0mm (press fit), length 10.0mm")
 		(tags "solder Pin_ press fit")
-		(property "Reference" "TP_TX2"
+		(property "Reference" "TX2"
 			(at 0.05 -1.4 0)
 			(layer "F.SilkS")
@@
 		(descr "LED SMD 0603 (1608 Metric), square (rectangular) end terminal, IPC-7351 nominal, (Body size source: http://www.tortai-tech.com/upload/download/2011102023233369053.pdf), generated with kicad-footprint-generator")
 		(tags "LED")
-		(property "Reference" "D_LED6"
-			(at -3.0625 0 0)
+		(property "Reference" "FC 2"
+			(at -3.37 0 0)
 			(layer "F.SilkS")
 			(effects
@@
 		(descr "solder Pin_ diameter 1.0mm, hole diameter 1.0mm (press fit), length 10.0mm")
 		(tags "solder Pin_ press fit")
-		(property "Reference" "TP_TX3"
+		(property "Reference" "TX3"
 			(at 0.05 -1.4 0)
 			(layer "F.SilkS")
@@
 		(descr "LED SMD 0603 (1608 Metric), square (rectangular) end terminal, IPC-7351 nominal, (Body size source: http://www.tortai-tech.com/upload/download/2011102023233369053.pdf), generated with kicad-footprint-generator")
 		(tags "LED")
-		(property "Reference" "D_LED3"
-			(at -3.3625 0 0)
+		(property "Reference" "3.3V"
+			(at -3.36 -0.05 0)
 			(layer "F.SilkS")
 			(effects
@@
 		(descr "LED SMD 0603 (1608 Metric), square (rectangular) end terminal, IPC-7351 nominal, (Body size source: http://www.tortai-tech.com/upload/download/2011102023233369053.pdf), generated with kicad-footprint-generator")
 		(tags "LED")
-		(property "Reference" "D_LED2"
+		(property "Reference" "10V"
 			(at -3.0625 0 0)
 			(layer "F.SilkS")
@@
 		(descr "solder Pin_ diameter 1.0mm, hole diameter 1.0mm (press fit), length 10.0mm")
 		(tags "solder Pin_ press fit")
-		(property "Reference" "TP_CC1"
+		(property "Reference" "CC"
 			(at 0.05 -1.4 0)
 			(layer "F.SilkS")
@@
 		(descr "solder Pin_ diameter 1.0mm, hole diameter 1.0mm (press fit), length 10.0mm")
 		(tags "solder Pin_ press fit")
-		(property "Reference" "TP_GND14"
+		(property "Reference" "GND"
 			(at 0.05 -1.4 0)
 			(layer "F.SilkS")
@@
 		(descr "solder Pin_ diameter 1.0mm, hole diameter 1.0mm (press fit), length 10.0mm")
 		(tags "solder Pin_ press fit")
-		(property "Reference" "TP_GND3"
+		(property "Reference" "GND"
 			(at -0.05 -1.4 0)
 			(layer "F.SilkS")
@@
 		(descr "solder Pin_ diameter 1.0mm, hole diameter 1.0mm (press fit), length 10.0mm")
 		(tags "solder Pin_ press fit")
-		(property "Reference" "TP_GND6"
+		(property "Reference" "GND"
 			(at 0.05 -1.4 0)
 			(layer "F.SilkS")
@@
 		(descr "solder Pin_ diameter 1.0mm, hole diameter 1.0mm (press fit), length 10.0mm")
 		(tags "solder Pin_ press fit")
-		(property "Reference" "TP_GND2"
+		(property "Reference" "GND"
 			(at 0.05 -1.4 0)
 			(layer "F.SilkS")
@@
 		(descr "solder Pin_ diameter 1.0mm, hole diameter 1.0mm (press fit), length 10.0mm")
 		(tags "solder Pin_ press fit")
-		(property "Reference" "TP_5V6"
+		(property "Reference" "5V"
 			(at 0.05 -1.4 0)
 			(layer "F.SilkS")
@@
 		(descr "solder Pin_ diameter 1.0mm, hole diameter 1.0mm (press fit), length 10.0mm")
 		(tags "solder Pin_ press fit")
-		(property "Reference" "TP_VTX1"
+		(property "Reference" "VTX"
 			(at 0.05 -1.4 0)
 			(layer "F.SilkS")
@@
 		(descr "solder Pin_ diameter 1.0mm, hole diameter 1.0mm (press fit), length 10.0mm")
 		(tags "solder Pin_ press fit")
-		(property "Reference" "TP_5V3"
+		(property "Reference" "5V"
 			(at -0.05 -1.4 0)
 			(layer "F.SilkS")
@@
 		(descr "solder Pin_ diameter 1.0mm, hole diameter 1.0mm (press fit), length 10.0mm")
 		(tags "solder Pin_ press fit")
-		(property "Reference" "TP_SDA1"
+		(property "Reference" "SDA"
 			(at 0.05 -1.4 0)
 			(layer "F.SilkS")
@@
 		(descr "LED SMD 0603 (1608 Metric), square (rectangular) end terminal, IPC-7351 nominal, (Body size source: http://www.tortai-tech.com/upload/download/2011102023233369053.pdf), generated with kicad-footprint-generator")
 		(tags "LED")
-		(property "Reference" "D_LED4"
-			(at -5.0625 -0.15 0)
+		(property "Reference" "3.3VG"
+			(at -3.82 -0.02 0)
 			(layer "F.SilkS")
 			(effects
@@
 		(descr "solder Pin_ diameter 1.0mm, hole diameter 1.0mm (press fit), length 10.0mm")
 		(tags "solder Pin_ press fit")
-		(property "Reference" "TP_RX2"
+		(property "Reference" "RX2"
 			(at 0.05 -1.4 0)
 			(layer "F.SilkS")
@@
 		(descr "LED SMD 0603 (1608 Metric), square (rectangular) end terminal, IPC-7351 nominal, (Body size source: http://www.tortai-tech.com/upload/download/2011102023233369053.pdf), generated with kicad-footprint-generator")
 		(tags "LED")
-		(property "Reference" "D_LED1"
+		(property "Reference" "5V"
 			(at -2.5625 0 0)
 			(layer "F.SilkS")
@@
 		(descr "solder Pin_ diameter 1.0mm, hole diameter 1.0mm (press fit), length 10.0mm")
 		(tags "solder Pin_ press fit")
-		(property "Reference" "TP_LED3"
+		(property "Reference" "LED"
 			(at 0.05 -1.4 0)
 			(layer "F.SilkS")
@@
 		(descr "solder Pin_ diameter 1.0mm, hole diameter 1.0mm (press fit), length 10.0mm")
 		(tags "solder Pin_ press fit")
-		(property "Reference" "TP_RX5"
+		(property "Reference" "RX5"
 			(at 0.05 -1.4 0)
 			(layer "F.SilkS")
@@
 		(descr "solder Pin_ diameter 1.0mm, hole diameter 1.0mm (press fit), length 10.0mm")
 		(tags "solder Pin_ press fit")
-		(property "Reference" "TP_5V2"
+		(property "Reference" "5V"
 			(at 0.05 -1.4 0)
 			(layer "F.SilkS")
@@
 		(descr "solder Pin_ diameter 1.0mm, hole diameter 1.0mm (press fit), length 10.0mm")
 		(tags "solder Pin_ press fit")
-		(property "Reference" "TP_GND7"
+		(property "Reference" "GND"
 			(at 0.05 -1.4 0)
 			(layer "F.SilkS")
@@
 		(descr "solder Pin_ diameter 1.0mm, hole diameter 1.0mm (press fit), length 10.0mm")
 		(tags "solder Pin_ press fit")
-		(property "Reference" "TP_RX3"
+		(property "Reference" "RX3"
 			(at 0.05 -1.4 0)
 			(layer "F.SilkS")
@@
 		(descr "LED SMD 0603 (1608 Metric), square (rectangular) end terminal, IPC-7351 nominal, (Body size source: http://www.tortai-tech.com/upload/download/2011102023233369053.pdf), generated with kicad-footprint-generator")
 		(tags "LED")
-		(property "Reference" "D_LED5"
-			(at -3.0625 0 0)
+		(property "Reference" "FC 1"
+			(at -3.39 0.01 0)
 			(layer "F.SilkS")
 			(effects
@@
 		(descr "solder Pin_ diameter 1.0mm, hole diameter 1.0mm (press fit), length 10.0mm")
 		(tags "solder Pin_ press fit")
-		(property "Reference" "TP_10V2"
+		(property "Reference" "10V"
 			(at 0.05 -1.4 0)
 			(layer "F.SilkS")
@@
 		(descr "solder Pin_ diameter 1.0mm, hole diameter 1.0mm (press fit), length 10.0mm")
 		(tags "solder Pin_ press fit")
-		(property "Reference" "TP_5V5"
+		(property "Reference" "5V"
 			(at 0.05 -1.4 0)
 			(layer "F.SilkS")
@@
 		(descr "solder Pin_ diameter 1.0mm, hole diameter 1.0mm (press fit), length 10.0mm")
 		(tags "solder Pin_ press fit")
-		(property "Reference" "TP_SCL1"
+		(property "Reference" "SCL"
 			(at 0.05 -1.4 0)
 			(layer "F.SilkS")
@@
 		(descr "solder Pin_ diameter 1.0mm, hole diameter 1.0mm (press fit), length 10.0mm")
 		(tags "solder Pin_ press fit")
-		(property "Reference" "TP_CAM1"
+		(property "Reference" "CAM"
 			(at 0.05 -1.4 0)
 			(layer "F.SilkS")
