File: Flight Controller.kicad_pcb (KiCad board)
At the start: 6 copper layers, 39.5 x 39.5 mm, 151 parts, among them IC2 AT7456E, J1 Conn_01x08_MountingPin, J2 USB_C_Receptacle_USB2.0_14P, Q2 BC817W, SW1 SW_SPST, U1 AT32F435RGT7, U2 LMR51430, U3 BMP280, U4 SPX3819M5-L-3-3, U5 LMR51430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

Commit message: Layout
Parts:
- removed C_DEC2: 100n, Capacitor_SMD:C_0402_1005Metric
- moved D2 18.7 mm to (142.6, 60.2)
- moved D_LED1 13.0 mm to (117.3, 72.3)
- moved D_LED2 13.0 mm to (117.3, 74.0)
- moved D_LED3 13.0 mm to (117.3, 75.8)
- moved D_LED4 13.0 mm to (117.3, 77.5)
- moved D_LED5 13.0 mm to (117.3, 68.8)
- moved D_LED6 13.0 mm to (117.3, 70.5)
- moved C_BARO2 4.23 mm to (135.2, 75.2)
- moved U3 4.23 mm to (137.1, 74.5)
- moved C_BARO1 4.23 mm to (136.7, 72.4)
- moved R_BUZ1 3.85 mm to (140.1, 76.9)
- moved C_DEC6 2.58 mm to (143.2, 77.7), turned to 0 degrees
- moved Y2 1.97 mm to (155.0, 86.7), turned to 90 degrees
- moved R_USB2 1.88 mm to (160.5, 76.0), turned to 0 degrees
- moved R_USB1 1.68 mm to (160.6, 91.2), turned to 0 degrees
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Connections:
- net Net-(U2-SW) renamed /SW5
Routing:
- net /OSD_SCLK: track 0.00 -> 25.1 mm, vias 0 -> 2
- net /OSD_MISO: track 0.00 -> 24.3 mm, vias 0 -> 2
- net /OSD_MOSI: track 0.00 -> 23.5 mm, vias 0 -> 2
- net +5V: track 0.00 -> 21.1 mm, vias 0 -> 7
- net /OSD_CS: track 0.00 -> 20.0 mm, vias 0 -> 2
- net GND: track 2.18 -> 17.8 mm, vias 10 -> 25
- net /VBAT+: track 13.5 -> 28.4 mm, vias 2 -> 4
- net /FLASH_CS: track 0.00 -> 13.4 mm, vias 0 -> 1
- net /FLASH_MISO: track 0.00 -> 12.1 mm, vias 0 -> 1
- net /BOOT: track 0.00 -> 10.9 mm
- net +3.3V: track 0.00 -> 10.5 mm
- net /FLASH_MOSI: track 0.00 -> 10.5 mm, vias 0 -> 1
- net /FLASH_SCLK: track 0.00 -> 10.1 mm, vias 0 -> 1
- net Net-(J2-CC1): track 0.00 -> 8.00 mm
- net Net-(J2-CC2): track 0.00 -> 7.72 mm
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- added copper zone on B.Cu, net +5V
- added copper zone on B.Cu, net /SW5
- added copper zone on B.Cu, net /VBAT+
- added copper zone on B.Cu, net GND

Commit message: Layout
Parts:
- moved D2 20.7 mm to (144.4, 80.8)
- moved C_DEC1 4.06 mm to (150.4, 84.6), turned to 90 degrees
- moved C_3V2 3.47 mm to (148.1, 82.5), turned to 0 degrees
- moved U4 2.35 mm to (145.9, 84.6), turned to 0 degrees
- moved C_3V1 1.86 mm to (148.8, 84.6), turned to 90 degrees
- moved C_3VG1 1.61 mm to (142.0, 87.9)
- moved U8 1.61 mm to (142.0, 85.0)
- moved C_3VG2 1.61 mm to (144.1, 87.1)
- moved Y1 1.07 mm to (137.4, 83.4)
Routing:
- net /5V_OUT: track 0.00 -> 4.19 mm
- net Net-(U4-BP): track 0.00 -> 1.37 mm
- net Net-(U8-BP): track 0.00 -> 1.37 mm
- net /RES1: track 3.24 -> 4.31 mm
- net /RES2: track 2.92 -> 4.00 mm
- net GND: track 17.8 -> 18.9 mm, vias 25 -> 32
- added copper zone on B.Cu, net +3.3V
- added copper zone on B.Cu, net +3.3V_GYRO
- added copper zone on B.Cu, net /5V_OUT

Commit message: Layout
Parts:
- moved G*** 30.9 mm to (132.9, 82.1)
- moved R_BOOT1 24.0 mm to (159.1, 96.5)
- moved G*** 22.7 mm to (133.1, 74.8)
- moved SW1 22.6 mm to (156.0, 94.2), turned to -90 degrees
- moved C_BARO2 22.4 mm to (140.5, 97.0), turned to 180 degrees
- moved C_BARO1 21.3 mm to (140.3, 93.4), turned to 0 degrees
- moved U3 21.1 mm to (141.2, 95.2), turned to 0 degrees
- moved C_GYRO1 20.5 mm to (151.3, 74.7)
- moved C_GYRO2 20.5 mm to (150.3, 74.7)
- moved U7 20.5 mm to (153.7, 76.0)
- moved C_GYRO3 20.5 mm to (154.1, 73.8)
- moved R_OSD2 18.3 mm to (153.8, 83.3), turned to 0 degrees
- moved R_OSD1 18.0 mm to (150.5, 83.1)
- moved C_OSD1 17.6 mm to (149.8, 70.6)
- moved C_OSD2 17.6 mm to (149.2, 80.6)
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Routing:
- net /S4: track 0.00 -> 24.6 mm, vias 0 -> 2
- net /S3: track 0.00 -> 23.0 mm, vias 0 -> 2
- net /GYRO_INT: track 0.00 -> 22.4 mm, vias 0 -> 2
- net /GYRO_MISO: track 0.00 -> 22.4 mm, vias 0 -> 2
- net /S1: track 0.00 -> 21.9 mm, vias 0 -> 2
- net /S2: track 0.00 -> 21.8 mm, vias 0 -> 2
- net GND: track 18.9 -> 40.2 mm, vias 32 -> 37
- net /VBAT+: track 28.4 -> 47.2 mm
- net /GYRO_SCLK: track 0.00 -> 18.5 mm
- net /FLASH_CS: track 13.4 -> 30.8 mm, vias 1 -> 3
- net /GYRO_CS: track 0.00 -> 17.3 mm
- net /GYRO_MOSI: track 0.00 -> 16.7 mm
- net /BARO_SDA: track 0.00 -> 16.0 mm
- net /BARO_SCL: track 0.00 -> 15.9 mm
- net /OSD_SCLK: track 25.1 -> 33.6 mm
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
Commit message: Layout
Routing:
- net GND: track 40.2 -> 50.5 mm, vias 37 -> 43
- net +5V: track 21.1 -> 24.6 mm
- net Net-(D_LED4-A): track 0.00 -> 1.76 mm, vias 0 -> 1
- net Net-(D_LED3-A): track 0.00 -> 1.76 mm, vias 0 -> 1
- net Net-(D_LED1-A): track 0.00 -> 1.76 mm, vias 0 -> 1
- net Net-(D_LED6-A): track 0.00 -> 1.72 mm, vias 0 -> 1
- net Net-(D_LED2-A): track 0.00 -> 1.72 mm, vias 0 -> 1
- net Net-(D_LED5-A): track 0.00 -> 1.62 mm, vias 0 -> 1

Commit message: Layout
Parts:
- moved R_I2C1 1.81 mm to (148.3, 95.1)
- moved R_I2C2 0.34 mm to (147.9, 92.3)
Routing:
- net /UART4_TX: track 0.00 -> 25.0 mm, vias 0 -> 2
- net /UART4_RX: track 0.00 -> 22.1 mm, vias 0 -> 2
- net /UART2_TX: track 1.72 -> 16.5 mm, vias 1 -> 2
- net /BOOT: track 5.15 -> 18.4 mm, vias 0 -> 2
- net /UART2_RX: track 1.84 -> 13.9 mm, vias 1 -> 2
- net /I2C2_SCL: track 3.63 -> 14.4 mm, vias 1 -> 2
- net /I2C2_SDA: track 5.00 -> 14.7 mm, vias 1 -> 2
- net /UART5_RX: track 0.00 -> 3.62 mm, vias 0 -> 2
- net /UART3_TX: track 1.40 -> 4.15 mm, vias 1 -> 2
- net +3.3V: track 16.9 -> 14.4 mm, vias 0 -> 2
- net GND: track 50.5 -> 48.1 mm
- net /UART5_TX: track 0.00 -> 2.46 mm, vias 0 -> 1
- net /UART3_RX: track 1.40 -> 3.35 mm, vias 1 -> 2
- net /S1: track 21.9 -> 23.2 mm
- net +10V: track 15.9 -> 16.6 mm
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